File: kicad working dir/espLite-a/espLite-a_relay/espLite-a_relay.sch (KiCad schematic (older format))
At the start: 14 parts

Commit message: work
Parts:
- added R?: R_Small_US, symbol Device:R_Small_US
Changed lines of the file:
@@
 Wire Wire Line
 	6800 4200 7200 4200
+$Comp
+L Device:R_Small_US R?
+U 1 1 5E317F08
+P 6300 4300
+F 0 "R?" H 6368 4346 50  0000 L CNN
+F 1 "R_Small_US" H 6368 4255 50  0000 L CNN
+F 2 "" H 6300 4300 50  0001 C CNN
+F 3 "~" H 6300 4300 50  0001 C CNN
+	1    6300 4300
+	1    0    0    -1
+$EndComp
 $EndSCHEMATC
